File: pcb_hw/Electronic Sculpture PCB rev1.sch (EAGLE design)
At the start: 28 parts, among them X1 CONNECTOR-2, X2 CONNECTOR-4, X3 CONNECTOR-4, X4 CONNECTOR-2

Commit message: added control buttons to the schematic
Parts:
- added JP5: (no value), HyTechDevices:M05
- added LIVE, PLAY, RECORD, RESET: BIG_PUSHBUTTON, 3872_Part_Library:BIG_PUSHBUTTON
- added ON/OFF_SWITCH: 0S102011MS2QS1, HyTechDevices:0S102011MS2QS1
- added R10, R11, R12, R13: (no value), HyTechDevices:RESISTORAXIAL-0.3
- added R14: (no value), HyTechDevices:3RP/1610N
Connections:
- new net BPM_CONTROL: JP5.1, R14.S
- new net LIVE_BTN: JP5.2, LIVE.S, LIVE.S1, R13.2
- new net N$1: ON/OFF_SWITCH.P, X1-1.S
- new net PLAY_BTN: JP5.3, PLAY.S, PLAY.S1, R12.2
- new net RECORD_BTN: JP5.4, R10.2, RECORD.S, RECORD.S1
- new net RESET_BTN: JP5.5, R11.2, RESET.S, RESET.S1
- net +12V: now also ON/OFF_SWITCH.S; no longer X1-1.S
- net +5V: now also R10.1, R11.1, R12.1, R13.1, R14.E
- net GND: now also LIVE.P, LIVE.P1, PLAY.P, PLAY.P1, R14.A, RECORD.P, RECORD.P1, RESET.P, RESET.P1
Other:
- note added: "BPM Control Potentiometer"
- note added: "Control Buttons"
- note added: "Control I/O"
- note added: "Pin A12 Pin A11 Pin A10 Pin A9 Pin A8"
- moved on the sheet: C11, JP1, JP2, JP3, JP4, MOTOR_CONTOLLER_1, MOTOR_CONTROLLER_2, R1, R2, R3, R4, R5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

Commit message: board design, gerbers
Parts:
- removed C3, C4: 10uF, HyTechDevices:CAPPTH1
- removed IC: LM386M-1, linear:LM386M-1
- removed JP3: M02, HyTechDevices:M02
- removed ON/OFF_SWITCH: 0S102011MS2QS1, HyTechDevices:0S102011MS2QS1
- removed R1, R14, R2, R3, R4, R5, R6, R7, R8, R9: (no value), HyTechDevices:3RP/1610N
- removed U$1: OKI-78SR-5, HyTechDevices:OKI-78SR-5
- removed X1: CONNECTOR-2, HyTechDevices:CONNECTOR-2
- added BPM_CONTROL, VOLUME: P0915N-QC20BR5K, 3872_Part_Library:P0915N-QC20BR5K
- added F1: 2A, HyTechDevices:FUSE_MINIBLADE
- added IC1: LM386N-1, linear:LM386N-1
- added MAIN_POWER: CONNECTOR-2, HyTechDevices:CONNECTOR-2
- added POWER: M04, HyTechDevices:M04
- added SLIDER_1, SLIDER_2, SLIDER_3, SLIDER_4, SLIDER_5, SLIDER_6, SLIDER_7, SLIDER_8: SLIDE_POT, 3872_Part_Library:SLIDE_POT
- CONTROLS: value (none) -> M05
- MOTOR_CONTROL, SEQUENCER_IO: value (none) -> M08
- R10, R11, R12, R13: value (none) -> 10k
- renumbered JP1 to SEQUENCER_IO, JP2 to MOTOR_CONTROL, JP4 to AUDIO, JP5 to CONTROLS, X2 to MOTOR1, X3 to MOTOR2, X4 to SPEAKER
Connections:
- removed net N$5: IC.+IN, R9.S
- new net N$2: C5.1, IC1.BYPASS
- net +12V: now also F1.2, IC1.VS, POWER.4; no longer C3.1, IC.VS, ON/OFF_SWITCH.S, U$1.IN
- net +5V: now also BPM_CONTROL.3, POWER.3, SLIDER_1.3, SLIDER_2.3, SLIDER_3.3, SLIDER_4.3, SLIDER_5.3, SLIDER_6.3, SLIDER_7.3, SLIDER_8.3; no longer C4.1, JP3.2, R1.E, R14.E, R2.E, R3.E, R4.E, R5.E, R6.E, R7.E, R8.E, U$1.OUT
- net AUDIO_OUT: now also VOLUME.3; no longer R9.E
- net BPM_CONTROL: now also BPM_CONTROL.2; no longer R14.S
- net GND: now also AUDIO.1, BPM_CONTROL.1, BPM_CONTROL.SHIELD, IC1.-IN, IC1.GND, MAIN_POWER-2.S, POWER.1, POWER.2, SLIDER_1.1, SLIDER_2.1, SLIDER_3.1, SLIDER_4.1, SLIDER_5.1, SLIDER_6.1, SLIDER_7.1, SLIDER_8.1, VOLUME.1, VOLUME.SHIELD; no longer C3.2, C4.2, IC.-IN, IC.GND, JP3.1, R1.A, R14.A, R2.A, R3.A, R4.A, R5.A, R6.A, R7.A, R8.A, R9.A, U$1.GND, X1-2.S
- net LIVE_BTN: now also CONTROLS.4; no longer CONTROLS.2
- net N$1: now also F1.1, MAIN_POWER-1.S; no longer ON/OFF_SWITCH.P, X1-1.S
- net N$3: now also IC1.+IN, VOLUME.2; no longer C5.1, IC.BYPASS
- net N$4: now also IC1.OUT; no longer IC.OUT
- net RECORD_BTN: now also CONTROLS.2; no longer CONTROLS.4
- net SLIDER_1: now also SLIDER_1.2; no longer R1.S
- net SLIDER_2: now also SLIDER_2.2; no longer R2.S
- net SLIDER_3: now also SLIDER_3.2; no longer R3.S
- net SLIDER_4: now also SLIDER_4.2; no longer R4.S
- net SLIDER_5: now also SLIDER_5.2; no longer R5.S
- net SLIDER_6: now also SLIDER_6.2; no longer R6.S
- net SLIDER_7: now also SLIDER_7.2; no longer R7.S
- net SLIDER_8: now also SLIDER_8.2; no longer R8.S
Other:
- note added: "Pin VIN Pin 5V Pin GND Pin GND"
- note added: "R15 Potentiometer works as a volume adjuster."
- note removed: "DC-DC Converter to convert 12V to 5V."
- note removed: "Pin VIN Pin GND"
- note removed: "R9 Potentiometer works as a volume adjuster."
- moved on the sheet: C11, C5, C6, C8, C9
